Commit message: chore: update package name and clean up

File: urdf/mecanum3.xacro (robot description, xacro)
@@ -1,12 +1,14 @@
 <?xml version="1.0" ?>
 <robot name="mecanum3" xmlns:xacro="http://www.ros.org/wiki/xacro">
-<xacro:include filename="$(find mecanum3_description)/urdf/materials.xacro" />
-<!-- <xacro:include filename="$(find mecanum3_description)/urdf/mecanum3.trans" />
-<xacro:include filename="$(find mecanum3_description)/urdf/mecanum3.gazebo" /> -->
+<xacro:include filename="$(find mecanumrover_description)/urdf/materials.xacro" />
+<!-- <xacro:include filename="$(find mecanumrover_description)/urdf/mecanum3.trans" /> -->
+<!-- <xacro:include filename="$(find mecanumrover_description)/urdf/mecanum3.gazebo" /> -->
+<!-- OPTION: LRF TG30 -->
+<xacro:include filename="$(find vs_rover_options_description)/urdf/lrf/tg30_mecanum3.xacro" />
 <link name="base_footprint" />
 <joint name="base_joint" type="fixed">
   <parent link="base_footprint"/>
   <child link="base_link" />
-  <origin xyz="0 0 0" rpy="0 0 -1.5708"/>
+  <origin xyz="0 0 0" rpy="0 0 ${radians(-90)}"/>
 </joint>
 <link name="base_link">
@@ -19,5 +21,5 @@
     <origin xyz="0 0 0" rpy="0 0 0"/>
     <geometry>
-      <mesh filename="package://mecanum3_description/meshes/base_link.stl" scale="0.001 0.001 0.001"/>
+      <mesh filename="package://mecanumrover_description/meshes/base_link.stl" scale="0.001 0.001 0.001"/>
     </geometry>
     <material name="silver"/>
@@ -26,5 +28,5 @@
     <origin xyz="0 0 0" rpy="0 0 0"/>
     <geometry>
-      <mesh filename="package://mecanum3_description/meshes/base_link.stl" scale="0.001 0.001 0.001"/>
+      <mesh filename="package://mecanumrover_description/meshes/base_link.stl" scale="0.001 0.001 0.001"/>
     </geometry>
   </collision>
@@ -39,12 +41,12 @@
     <origin xyz="0.0875 -0.12 -0.076" rpy="0 0 0"/>
     <geometry>
-      <mesh filename="package://mecanum3_description/meshes/front_left_wheel_1.stl" scale="0.001 0.001 0.001"/>
+      <mesh filename="package://mecanumrover_description/meshes/front_left_wheel_1.stl" scale="0.001 0.001 0.001"/>
     </geometry>
-    <material name="silver"/>
+    <material name="dark_grey"/>
   </visual>
   <collision>
     <origin xyz="0.0875 -0.12 -0.076" rpy="0 0 0"/>
     <geometry>
-      <mesh filename="package://mecanum3_description/meshes/front_left_wheel_1.stl" scale="0.001 0.001 0.001"/>
+      <mesh filename="package://mecanumrover_description/meshes/front_left_wheel_1.stl" scale="0.001 0.001 0.001"/>
     </geometry>
   </collision>
@@ -59,12 +61,12 @@
     <origin xyz="-0.0875 -0.12 -0.076" rpy="0 0 0"/>
     <geometry>
-      <mesh filename="package://mecanum3_description/meshes/front_right_wheel_1.stl" scale="0.001 0.001 0.001"/>
+      <mesh filename="package://mecanumrover_description/meshes/front_right_wheel_1.stl" scale="0.001 0.001 0.001"/>
     </geometry>
-    <material name="silver"/>
+    <material name="dark_grey"/>
   </visual>
   <collision>
     <origin xyz="-0.0875 -0.12 -0.076" rpy="0 0 0"/>
     <geometry>
-      <mesh filename="package://mecanum3_description/meshes/front_right_wheel_1.stl" scale="0.001 0.001 0.001"/>
+      <mesh filename="package://mecanumrover_description/meshes/front_right_wheel_1.stl" scale="0.001 0.001 0.001"/>
     </geometry>
   </collision>
@@ -79,12 +81,12 @@
     <origin xyz="-0.0875 0.12 -0.076" rpy="0 0 0"/>
     <geometry>
-      <mesh filename="package://mecanum3_description/meshes/back_right_wheel_1.stl" scale="0.001 0.001 0.001"/>
+      <mesh filename="package://mecanumrover_description/meshes/back_right_wheel_1.stl" scale="0.001 0.001 0.001"/>
     </geometry>
-    <material name="silver"/>
+    <material name="dark_grey"/>
   </visual>
   <collision>
     <origin xyz="-0.0875 0.12 -0.076" rpy="0 0 0"/>
     <geometry>
-      <mesh filename="package://mecanum3_description/meshes/back_right_wheel_1.stl" scale="0.001 0.001 0.001"/>
+      <mesh filename="package://mecanumrover_description/meshes/back_right_wheel_1.stl" scale="0.001 0.001 0.001"/>
     </geometry>
   </collision>
@@ -99,12 +101,12 @@
     <origin xyz="0.0875 0.12 -0.076" rpy="0 0 0"/>
     <geometry>
-      <mesh filename="package://mecanum3_description/meshes/back_left_wheel_1.stl" scale="0.001 0.001 0.001"/>
+      <mesh filename="package://mecanumrover_description/meshes/back_left_wheel_1.stl" scale="0.001 0.001 0.001"/>
     </geometry>
-    <material name="silver"/>
+    <material name="dark_grey"/>
   </visual>
   <collision>
     <origin xyz="0.0875 0.12 -0.076" rpy="0 0 0"/>
     <geometry>
-      <mesh filename="package://mecanum3_description/meshes/back_left_wheel_1.stl" scale="0.001 0.001 0.001"/>
+      <mesh filename="package://mecanumrover_description/meshes/back_left_wheel_1.stl" scale="0.001 0.001 0.001"/>
     </geometry>
   </collision>
