Commit message: Restore original mecanumrover_description tree

File: urdf/materials.xacro (robot description, xacro)
@@ -13,3 +13,6 @@
     <color rgba="0.100 0.100 0.100 1.000" />
   </material>
+  <material name="cream">
+    <color rgba="0.9725 0.8941 0.6941 1.0" />
+  </material>
 </robot>

File: urdf/mecanum3.xacro (robot description, xacro)
@@ -1,138 +1,270 @@
 <?xml version="1.0" ?>
 <robot name="mecanum3" xmlns:xacro="http://www.ros.org/wiki/xacro">
-<xacro:include filename="$(find mecanumrover_description)/urdf/materials.xacro" />
-<!-- <xacro:include filename="$(find mecanumrover_description)/urdf/mecanum3.trans" /> -->
-<!-- <xacro:include filename="$(find mecanumrover_description)/urdf/mecanum3.gazebo" /> -->
-<!-- OPTION: LRF TG30 -->
-<xacro:include filename="$(find vs_rover_options_description)/urdf/lrf/tg30_mecanum3.xacro" />
-<link name="base_footprint" />
-<joint name="base_joint" type="fixed">
-  <parent link="base_footprint"/>
-  <child link="base_link" />
-  <origin xyz="0 0 0" rpy="0 0 ${radians(-90)}"/>
-</joint>
-<link name="base_link">
-  <inertial>
-    <origin xyz="8.039076182406018e-05 -0.001484050423595346 0.11040223412633365" rpy="0 0 0"/>
-    <mass value="51.54953324093924"/>
-    <inertia ixx="0.451406" iyy="0.211369" izz="0.557559" ixy="0.000784" iyz="0.000199" ixz="-0.000134"/>
-  </inertial>
-  <visual>
-    <origin xyz="0 0 0" rpy="0 0 0"/>
-    <geometry>
-      <mesh filename="package://mecanumrover_description/meshes/base_link.stl" scale="0.001 0.001 0.001"/>
-    </geometry>
-    <material name="silver"/>
-  </visual>
-  <collision>
-    <origin xyz="0 0 0" rpy="0 0 0"/>
-    <geometry>
-      <mesh filename="package://mecanumrover_description/meshes/base_link.stl" scale="0.001 0.001 0.001"/>
-    </geometry>
-  </collision>
-</link>
-<link name="front_left_wheel_1">
-  <inertial>
-    <origin xyz="-0.03247844667661433 -1.7208456881689926e-15 1.3877787807814457e-17" rpy="0 0 0"/>
-    <mass value="6.210672529256712"/>
-    <inertia ixx="0.017207" iyy="0.009618" izz="0.009618" ixy="0.0" iyz="0.0" ixz="-0.0"/>
-  </inertial>
-  <visual>
-    <origin xyz="0.0875 -0.12 -0.076" rpy="0 0 0"/>
-    <geometry>
-      <mesh filename="package://mecanumrover_description/meshes/front_left_wheel_1.stl" scale="0.001 0.001 0.001"/>
-    </geometry>
-    <material name="dark_grey"/>
-  </visual>
-  <collision>
-    <origin xyz="0.0875 -0.12 -0.076" rpy="0 0 0"/>
-    <geometry>
-      <mesh filename="package://mecanumrover_description/meshes/front_left_wheel_1.stl" scale="0.001 0.001 0.001"/>
-    </geometry>
-  </collision>
-</link>
-<link name="front_right_wheel_1">
-  <inertial>
-    <origin xyz="0.032478446676614314 -3.7470027081099033e-16 1.3877787807814457e-17" rpy="0 0 0"/>
-    <mass value="6.210672529256714"/>
-    <inertia ixx="0.017207" iyy="0.009618" izz="0.009618" ixy="-0.0" iyz="0.0" ixz="0.0"/>
-  </inertial>
-  <visual>
-    <origin xyz="-0.0875 -0.12 -0.076" rpy="0 0 0"/>
-    <geometry>
-      <mesh filename="package://mecanumrover_description/meshes/front_right_wheel_1.stl" scale="0.001 0.001 0.001"/>
-    </geometry>
-    <material name="dark_grey"/>
-  </visual>
-  <collision>
-    <origin xyz="-0.0875 -0.12 -0.076" rpy="0 0 0"/>
-    <geometry>
-      <mesh filename="package://mecanumrover_description/meshes/front_right_wheel_1.stl" scale="0.001 0.001 0.001"/>
-    </geometry>
-  </collision>
-</link>
-<link name="back_right_wheel_1">
-  <inertial>
-    <origin xyz="0.03247844667661433 1.7208456881689926e-15 1.3877787807814457e-17" rpy="0 0 0"/>
-    <mass value="6.210672529256712"/>
-    <inertia ixx="0.017207" iyy="0.009618" izz="0.009618" ixy="0.0" iyz="0.0" ixz="0.0"/>
-  </inertial>
-  <visual>
-    <origin xyz="-0.0875 0.12 -0.076" rpy="0 0 0"/>
-    <geometry>
-      <mesh filename="package://mecanumrover_description/meshes/back_right_wheel_1.stl" scale="0.001 0.001 0.001"/>
-    </geometry>
-    <material name="dark_grey"/>
-  </visual>
-  <collision>
-    <origin xyz="-0.0875 0.12 -0.076" rpy="0 0 0"/>
-    <geometry>
-      <mesh filename="package://mecanumrover_description/meshes/back_right_wheel_1.stl" scale="0.001 0.001 0.001"/>
-    </geometry>
-  </collision>
-</link>
-<link name="back_left_wheel_1">
-  <inertial>
-    <origin xyz="-0.03247844667661433 3.7470027081099033e-16 0.0" rpy="0 0 0"/>
-    <mass value="6.210672529256715"/>
-    <inertia ixx="0.017207" iyy="0.009618" izz="0.009618" ixy="-0.0" iyz="0.0" ixz="0.0"/>
-  </inertial>
-  <visual>
-    <origin xyz="0.0875 0.12 -0.076" rpy="0 0 0"/>
-    <geometry>
-      <mesh filename="package://mecanumrover_description/meshes/back_left_wheel_1.stl" scale="0.001 0.001 0.001"/>
-    </geometry>
-    <material name="dark_grey"/>
-  </visual>
-  <collision>
-    <origin xyz="0.0875 0.12 -0.076" rpy="0 0 0"/>
-    <geometry>
-      <mesh filename="package://mecanumrover_description/meshes/back_left_wheel_1.stl" scale="0.001 0.001 0.001"/>
-    </geometry>
-  </collision>
-</link>
-<joint name="front_left_joint" type="continuous">
-  <origin xyz="-0.0875 0.12 0.076" rpy="0 0 0"/>
-  <parent link="base_link"/>
-  <child link="front_left_wheel_1"/>
-  <axis xyz="-1.0 0.0 0.0"/>
-</joint>
-<joint name="front_right_joint" type="continuous">
-  <origin xyz="0.0875 0.12 0.076" rpy="0 0 0"/>
-  <parent link="base_link"/>
-  <child link="front_right_wheel_1"/>
-  <axis xyz="1.0 0.0 0.0"/>
-</joint>
-<joint name="back_right_joint" type="continuous">
-  <origin xyz="0.0875 -0.12 0.076" rpy="0 0 0"/>
-  <parent link="base_link"/>
-  <child link="back_right_wheel_1"/>
-  <axis xyz="1.0 0.0 0.0"/>
-</joint>
-<joint name="back_left_joint" type="continuous">
-  <origin xyz="-0.0875 -0.12 0.076" rpy="0 0 0"/>
-  <parent link="base_link"/>
-  <child link="back_left_wheel_1"/>
-  <axis xyz="-1.0 0.0 0.0"/>
-</joint>
+  <xacro:include filename="$(find mecanumrover_description)/urdf/materials.xacro" />
+  <xacro:include filename="$(find mecanumrover_description)/urdf/mecanum3.gazebo" />
+  <xacro:include filename="$(find mecanumrover_description)/urdf/mecanum3_ros2_control.xacro" />
+  <!-- OPTION LRF TG30 -->
+  <!--<xacro:include filename="$(find vs_rover_options_description)/urdf/lrf/tg30_mecanum3.xacro" />-->
+  <!-- Inertial macros -->
+  <xacro:macro name="cylinder_inertial" params="mass radius length">
+    <mass value="${mass}"/>
+    <inertia
+      ixx="${((radius*radius)/4 + (length*length)/12)*mass}"
+      ixy="0" ixz="0"
+      iyy="${((radius*radius)/4 + (length*length)/12)*mass}"
+      iyz="0"
+      izz="${(mass*radius*radius)/2}" />
+  </xacro:macro>
+  <!-- Barrel (roller) macros  -->
+  <xacro:macro name="barrel_rl" params="prefix parent dir rot">
+    <joint name="${prefix}_joint" type="continuous">
+      <parent link="${parent}"/>
+      <child  link="${prefix}_link"/>
+      <origin
+        xyz="${0.0666389*cos(radians(dir))} ${0.0666389*sin(radians(dir))} 0"
+        rpy="${pi/4*rot} 0 ${radians(dir)}"/>
+      <axis xyz="0 0 1"/>
+      <dynamics damping="0.001" friction="0.0"/>
+    </joint>
+    <link name="${prefix}_link">
+      <visual>
+        <geometry>
+          <mesh filename="package://mecanumrover_description/meshes/mecanum3/mecanum_barrel.stl"/>
+        </geometry>
+        <material name="dark_grey"/>
+      </visual>
+      <collision>
+        <geometry>
+          <mesh filename="package://mecanumrover_description/meshes/mecanum3/mecanum_barrel.stl"/>
+        </geometry>
+      </collision>
+      <inertial>
+        <xacro:cylinder_inertial
+          mass="0.01225"
+          radius="0.00956"
+          length="0.0381"/>
+      </inertial>
+    </link>
+  </xacro:macro>
+  <xacro:macro name="barrels_rl" params="prefix parent rot">
+    <xacro:barrel_rl prefix="${prefix}_0"  parent="${parent}" dir="0"   rot="${rot}"/>
+    <xacro:barrel_rl prefix="${prefix}_1"  parent="${parent}" dir="24"  rot="${rot}"/>
+    <xacro:barrel_rl prefix="${prefix}_2"  parent="${parent}" dir="48"  rot="${rot}"/>
+    <xacro:barrel_rl prefix="${prefix}_3"  parent="${parent}" dir="72"  rot="${rot}"/>
+    <xacro:barrel_rl prefix="${prefix}_4"  parent="${parent}" dir="96"  rot="${rot}"/>
+    <xacro:barrel_rl prefix="${prefix}_5"  parent="${parent}" dir="120" rot="${rot}"/>
+    <xacro:barrel_rl prefix="${prefix}_6"  parent="${parent}" dir="144" rot="${rot}"/>
+    <xacro:barrel_rl prefix="${prefix}_7"  parent="${parent}" dir="168" rot="${rot}"/>
+    <xacro:barrel_rl prefix="${prefix}_8"  parent="${parent}" dir="192" rot="${rot}"/>
+    <xacro:barrel_rl prefix="${prefix}_9"  parent="${parent}" dir="216" rot="${rot}"/>
+    <xacro:barrel_rl prefix="${prefix}_10" parent="${parent}" dir="240" rot="${rot}"/>
+    <xacro:barrel_rl prefix="${prefix}_11" parent="${parent}" dir="264" rot="${rot}"/>
+    <xacro:barrel_rl prefix="${prefix}_12" parent="${parent}" dir="288" rot="${rot}"/>
+    <xacro:barrel_rl prefix="${prefix}_13" parent="${parent}" dir="312" rot="${rot}"/>
+    <xacro:barrel_rl prefix="${prefix}_14" parent="${parent}" dir="336" rot="${rot}"/>
+  </xacro:macro>
+  <xacro:macro name="attach_mecanum_rollers" params="wheel_prefix wheel_link rot">
+    <xacro:barrels_rl
+      prefix="${wheel_prefix}_barrel"
+      parent="${wheel_link}"
+      rot="${rot}"/>
+  </xacro:macro>
+  <!-- Base -->
+  <link name="base_footprint"/>
+  <joint name="base_joint" type="fixed">
+    <parent link="base_footprint"/>
+    <child link="base_link"/>
+    <origin xyz="0 0 0" rpy="0 0 -1.5708"/>
+  </joint>
+  <link name="base_link">
+    <inertial>
+      <origin xyz="0.000129 -0.001817 0.110883"/>
+      <mass value="14"/>
+      <inertia ixx="1.346868e-01" iyy="4.468661e-02" izz="1.499091e-01" ixy="3.076527e-04" ixz="-2.931603e-05" iyz="2.763693e-05"/>
+    </inertial>
+    <visual>
+      <geometry>
+        <mesh filename="package://mecanumrover_description/meshes/mecanum3/base_link.stl"
+              scale="0.001 0.001 0.001"/>
+      </geometry>
+      <material name="silver"/>
+    </visual>
+    <collision>
+      <geometry>
+        <mesh filename="package://mecanumrover_description/meshes/mecanum3/base_link.stl"
+              scale="0.001 0.001 0.001"/>
+      </geometry>
+    </collision>
+  </link>
+  <!-- Arm link macro -->
+  <xacro:macro name="mecanum_arm_link" params="name">
+    <link name="${name}">
+      <inertial>
+        <origin xyz="0.001000 -0.054014 1.236051e-21"/>
+        <mass value="0.5"/>
+        <inertia ixx="7.442105e-04" iyy="2.141603e-04" izz="5.341336e-04" ixy="-4.944204e-21" ixz="1.236051e-21" iyz="1.089631e-04"/>
+      </inertial>
+      <visual>
+        <geometry>
+          <mesh filename="package://mecanumrover_description/meshes/mecanum3/arms.stl"
+                scale="0.001 0.001 0.001"/>
+        </geometry>
+        <material name="silver"/>
+      </visual>
+      <collision>
+        <geometry>
+          <mesh filename="package://mecanumrover_description/meshes/mecanum3/arms.stl"
+                scale="0.001 0.001 0.001"/>
+        </geometry>
+      </collision>
+    </link>
+  </xacro:macro>
+  <!-- Suspension joint macro -->
+  <xacro:macro name="mecanum_suspension_joint"
+               params="name parent child xyz rpy">
+    <joint name="${name}" type="revolute">
+      <parent link="${parent}"/>
+      <child link="${child}"/>
+      <origin xyz="${xyz}" rpy="${rpy}"/>
+      <axis xyz="1 0 0"/>
+      <limit lower="-0.10472" upper="0" effort="300" velocity="20"/>
+      <dynamics damping="5.0" friction="0.1"/>
+    </joint>
+  </xacro:macro>
+  <!-- Wheel link macros -->
+  <xacro:macro name="mecanum_wheel_link" params="name">
+    <link name="${name}">
+      <inertial>
+        <origin xyz="0 0 0"/>
+        <mass value="0.88"/>
+        <inertia ixx="7.666816e-04" iyy="7.666974e-04" izz="8.946765e-04" ixy="2.614197e-11" ixz="1.015151e-09" iyz="-2.439097e-09"/>
+      </inertial>
+      <visual>
+        <geometry>
+          <mesh filename="package://mecanumrover_description/meshes/mecanum3/mecanum_wheel.stl"
+                scale="0.001 0.001 0.001"/>
+        </geometry>
+        <material name="silver"/>
+      </visual>
+      <collision>
+        <geometry>
+          <mesh filename="package://mecanumrover_description/meshes/mecanum3/mecanum_wheel.stl"
+                scale="0.001 0.001 0.001"/>
+        </geometry>
+      </collision>
+    </link>
+  </xacro:macro>
+  <xacro:macro name="mecanum_wheel_rev_link" params="name">
+    <link name="${name}">
+      <inertial>
+        <origin xyz="0.000657 0 0.007742"/>
+        <mass value="0.88"/>
+        <inertia ixx="7.655818e-04" iyy="7.655769e-04" izz="8.900386e-04" ixy="-6.106217e-09" ixz="1.064093e-09" iyz="-2.991811e-09"/>
+      </inertial>
+      <visual>
+        <geometry>
+          <mesh filename="package://mecanumrover_description/meshes/mecanum3/mecanum_wheel_rev.stl"
+                scale="0.001 0.001 0.001"/>
+        </geometry>
+        <material name="silver"/>
+      </visual>
+      <collision>
+        <geometry>
+          <mesh filename="package://mecanumrover_description/meshes/mecanum3/mecanum_wheel_rev.stl"
+                scale="0.001 0.001 0.001"/>
+        </geometry>
+      </collision>
+    </link>
+  </xacro:macro>
+  <!-- Wheel joint macro -->
+  <xacro:macro name="mecanum_wheel_joint"
+               params="name parent child xyz rpy axis_z">
+    <joint name="${name}" type="continuous">
+      <parent link="${parent}"/>
+      <child link="${child}"/>
+      <origin xyz="${xyz}" rpy="${rpy}"/>
+      <axis xyz="0 0 ${axis_z}"/>
+    </joint>
+  </xacro:macro>
+  <!-- Arms -->
+  <xacro:mecanum_arm_link name="front_left_arm"/>
+  <xacro:mecanum_arm_link name="front_right_arm"/>
+  <xacro:mecanum_arm_link name="back_left_arm"/>
+  <xacro:mecanum_arm_link name="back_right_arm"/>
+  <!-- Suspension joints -->
+  <xacro:mecanum_suspension_joint
+    name="front_left_suspension_joint"
+    parent="base_link"
+    child="front_left_arm"
+    xyz="-0.085 0.020 0.076"
+    rpy="0 0 ${radians(180)}"/>
+  <xacro:mecanum_suspension_joint
+    name="front_right_suspension_joint"
+    parent="base_link"
+    child="front_right_arm"
+    xyz="0.085 0.020 0.076"
+    rpy="0 0 ${radians(180)}"/>
+  <xacro:mecanum_suspension_joint
+    name="back_left_suspension_joint"
+    parent="base_link"
+    child="back_left_arm"
+    xyz="-0.085 -0.020 0.076"
+    rpy="0 0 0"/>
+  <xacro:mecanum_suspension_joint
+    name="back_right_suspension_joint"
+    parent="base_link"
+    child="back_right_arm"
+    xyz="0.085 -0.020 0.076"
+    rpy="0 0 0"/>
+  <!-- Wheels -->
+  <xacro:mecanum_wheel_rev_link name="front_left_wheel_1"/>
+  <xacro:mecanum_wheel_link     name="front_right_wheel_1"/>
+  <xacro:mecanum_wheel_link     name="back_left_wheel_1"/>
+  <xacro:mecanum_wheel_rev_link name="back_right_wheel_1"/>
+  <!-- Wheel joints -->
+  <xacro:mecanum_wheel_joint
+    name="front_left_joint"
+    parent="front_left_arm"
+    child="front_left_wheel_1"
+    xyz="0.03 -0.100 0"
+    rpy="0 ${radians(-270)} 0"
+    axis_z="-1"/>
+  <xacro:mecanum_wheel_joint
+    name="front_right_joint"
+    parent="front_right_arm"
+    child="front_right_wheel_1"
+    xyz="-0.03 -0.100 0"
+    rpy="0 ${radians(-90)} 0"
+    axis_z="1"/>
+  <xacro:mecanum_wheel_joint
+    name="back_left_joint"
+    parent="back_left_arm"
+    child="back_left_wheel_1"
+    xyz="-0.03 -0.100 0"
+    rpy="0 ${radians(270)} 0"
+    axis_z="-1"/>
+  <xacro:mecanum_wheel_joint
+    name="back_right_joint"
+    parent="back_right_arm"
+    child="back_right_wheel_1"
+    xyz="0.03 -0.100 0"
+    rpy="0 ${radians(90)} 0"
+    axis_z="1"/>
+  <!-- Attach mecanum rollers -->
+  <xacro:attach_mecanum_rollers
+    wheel_prefix="front_left"
+    wheel_link="front_left_wheel_1"
+    rot="-1"/>
+  <xacro:attach_mecanum_rollers
+    wheel_prefix="back_left"
+    wheel_link="back_left_wheel_1"
+    rot="1"/>
+  <xacro:attach_mecanum_rollers
+    wheel_prefix="front_right"
+    wheel_link="front_right_wheel_1"
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