Commit message: xacro/urdfの修正

File: urdf/g120a.xacro (robot description, xacro)
@@ -1,9 +1,12 @@
 <?xml version="1.0" ?>
 <robot name="g120a" xmlns:xacro="http://www.ros.org/wiki/xacro">
+  <xacro:arg name="use_ros2_control" default="true" />
   <xacro:include filename="$(find mecanumrover_description)/urdf/materials.xacro" />
   <xacro:include filename="$(find mecanumrover_description)/urdf/g120a.gazebo" />
   <xacro:include filename="$(find vs_rover_options_description)/urdf/lrf/tg30_g120a.xacro" />
   <!-- OPTION LRF TG30 -->
-  <!--<xacro:include filename="$(find mecanumrover_description)/urdf/g120a_ros2_control.xacro" />-->
+  <!-- <xacro:if value="$(arg use_ros2_control)">
+    <xacro:include filename="$(find mecanumrover_description)/urdf/g120a_ros2_control.xacro" />
+  </xacro:if>-->
   <!-- Inertial macros -->
   <xacro:macro name="cylinder_inertial" params="mass radius length">
@@ -71,13 +74,14 @@
     <parent link="base_footprint"/>
     <child link="base_link"/>
-    <origin xyz="0 0 0.045" rpy="0 0 -1.5708"/>
+    <origin xyz="0 0 0.045" rpy="0 0 0"/>
   </joint>
   <link name="base_link">
     <inertial>
-      <origin xyz="0.00008 -0.001484 0.05"/>
+      <origin xyz="-0.001484 -0.00008 0.05"/>
       <mass value="35.6"/>
-      <inertia ixx="5.260826e-01" iyy="2.253078e-01" izz="6.264345e-01" ixy="-6.578214e-11" iyz="4.340698e-04" ixz="7.274235e-12"/>
+      <inertia ixx="2.253078e-01" iyy="5.260826e-01" izz="6.264345e-01" ixy="6.578214e-11" iyz="-7.274235e-12" ixz="4.340698e-04"/>
     </inertial>
     <visual>
+      <origin xyz="0 0 0" rpy="0 0 -1.5708"/>
       <geometry>
         <mesh filename="package://mecanumrover_description/meshes/g120a/base_link.stl"
@@ -87,4 +91,5 @@
     </visual>
     <collision>
+      <origin xyz="0 0 0" rpy="0 0 -1.5708"/>
       <geometry>
         <mesh filename="package://mecanumrover_description/meshes/g120a/base_link.stl"
@@ -193,24 +198,24 @@
     parent="base_link"
     child="front_left_arm"
-    xyz="-0.119 0.035 0.058"
-    rpy="0.0610865 0 ${radians(180)}"/>
+    xyz="0.035 0.119 0.058"
+    rpy="0.0610865 0 ${radians(90)}"/>
   <xacro:g120a_suspension_joint
     name="front_right_suspension_joint"
     parent="base_link"
     child="front_right_arm"
-    xyz="0.119 0.035 0.058"
-    rpy="0.0610865 0 ${radians(180)}"/>
+    xyz="0.035 -0.119 0.058"
+    rpy="0.0610865 0 ${radians(90)}"/>
   <xacro:g120a_suspension_joint
     name="back_left_suspension_joint"
     parent="base_link"
     child="back_left_arm"
-    xyz="-0.119 -0.035 0.058"
-    rpy="0.0610865 0 0"/>
+    xyz="-0.035 0.119 0.058"
+    rpy="0.0610865 0 ${radians(-90)}"/>
   <xacro:g120a_suspension_joint
     name="back_right_suspension_joint"
     parent="base_link"
     child="back_right_arm"
-    xyz="0.119 -0.035 0.058"
-    rpy="0.0610865 0 0"/>
+    xyz="-0.035 -0.119 0.058"
+    rpy="0.0610865 0 ${radians(-90)}"/>
   <!-- Wheels -->
   <xacro:g120a_wheel_rev_link name="front_left_wheel_1"/>

File: urdf/g40a_lb.xacro (robot description, xacro)
@@ -1,7 +1,10 @@
 <?xml version="1.0" ?>
 <robot name="g40a_lb" xmlns:xacro="http://www.ros.org/wiki/xacro">
+  <xacro:arg name="use_ros2_control" default="true" />
   <xacro:include filename="$(find mecanumrover_description)/urdf/materials.xacro" />
   <xacro:include filename="$(find mecanumrover_description)/urdf/g40a_lb.gazebo" />
-  <xacro:include filename="$(find mecanumrover_description)/urdf/g40a_lb_ros2_control.xacro" />
+  <xacro:if value="$(arg use_ros2_control)">
+    <xacro:include filename="$(find mecanumrover_description)/urdf/g40a_lb_ros2_control.xacro" />
+  </xacro:if>
   <!-- OPTION LRF TG30 -->
   <!--<xacro:include filename="$(find vs_rover_options_description)/urdf/lrf/tg30_g40a_lb.xacro" />-->
@@ -75,5 +78,5 @@
     <parent link="base_footprint"/>
     <child link="base_link"/>
-    <origin xyz="0 0 0" rpy="0 0 -1.5708"/>
+    <origin xyz="0 0 0" rpy="0 0 0"/>
   </joint>
   <link name="base_link">
@@ -82,8 +85,9 @@
       <mass value="20.75"/>
       <inertia
-        ixx="3.024773e-01" iyy="1.757975e-01" izz="2.820812e-01"
-        ixy="2.259609e-03" iyz="2.509410e-03" ixz="-6.536919e-04"/>
+        ixx="1.757975e-01" iyy="3.024773e-01" izz="2.820812e-01"
+        ixy="-2.259609e-03" iyz="6.536919e-04" ixz="2.509410e-03"/>
     </inertial>
     <visual>
+      <origin xyz="0 0 0" rpy="0 0 -1.5708"/>
       <geometry>
         <mesh filename="package://mecanumrover_description/meshes/g40a_lb/base_link.stl"
@@ -93,4 +97,5 @@
     </visual>
     <collision>
+      <origin xyz="0 0 0" rpy="0 0 -1.5708"/>
       <geometry>
         <mesh filename="package://mecanumrover_description/meshes/g40a_lb/base_link.stl"
@@ -139,10 +144,10 @@
     parent="base_link"
     child="front_lrf_mount"
-    xyz="0.0 0.0 0.0" rpy="0 0 ${radians(0)}"/>
+    xyz="0.0 0.0 0.0" rpy="0 0 ${radians(-90)}"/>
     <xacro:mecanum_lrf_mount
     name="back_lrf_mount"
     parent="base_link"
     child="back_lrf_mount"
-    xyz="0.0 0.0 0.0" rpy="0 0 ${radians(180)}"/>
+    xyz="0.0 0.0 0.0" rpy="0 0 ${radians(90)}"/>
   <!-- Arm link macro -->
   <xacro:macro name="mecanum_arm_link" params="name">
@@ -253,24 +258,24 @@
     parent="base_link"
     child="front_left_arm"
-    xyz="-0.1179 0.020 0.076"
-    rpy="0 0 ${radians(180)}"/>
+    xyz="0.020 0.1179 0.076"
+    rpy="0 0 ${radians(90)}"/>
   <xacro:mecanum_suspension_joint
     name="front_right_suspension_joint"
     parent="base_link"
     child="front_right_arm"
-    xyz="0.1179 0.020 0.076"
-    rpy="0 0 ${radians(180)}"/>
+    xyz="0.020 -0.1179 0.076"
+    rpy="0 0 ${radians(90)}"/>
   <xacro:mecanum_suspension_joint
     name="back_left_suspension_joint"
     parent="base_link"
     child="back_left_arm"
-    xyz="-0.1179 -0.020 0.076"
-    rpy="0 0 0"/>
+    xyz="-0.020 0.1179 0.076"
+    rpy="0 0 ${radians(-90)}"/>
   <xacro:mecanum_suspension_joint
     name="back_right_suspension_joint"
     parent="base_link"
     child="back_right_arm"
-    xyz="0.1179 -0.020 0.076"
-    rpy="0 0 0"/>
+    xyz="-0.020 -0.1179 0.076"
+    rpy="0 0 ${radians(-90)}"/>
   <!-- Wheels -->
   <xacro:mecanum_wheel_rev_link name="front_left_wheel_1"/>

File: urdf/mecanum3.xacro (robot description, xacro)
@@ -1,7 +1,10 @@
 <?xml version="1.0" ?>
 <robot name="mecanum3" xmlns:xacro="http://www.ros.org/wiki/xacro">
+  <xacro:arg name="use_ros2_control" default="true" />
   <xacro:include filename="$(find mecanumrover_description)/urdf/materials.xacro" />
   <xacro:include filename="$(find mecanumrover_description)/urdf/mecanum3.gazebo" />
-  <xacro:include filename="$(find mecanumrover_description)/urdf/mecanum3_ros2_control.xacro" />
+  <xacro:if value="$(arg use_ros2_control)">
+    <xacro:include filename="$(find mecanumrover_description)/urdf/mecanum3_ros2_control.xacro" />
+  </xacro:if>
   <!-- OPTION LRF TG30 -->
   <!--<xacro:include filename="$(find vs_rover_options_description)/urdf/lrf/tg30_mecanum3.xacro" />-->
@@ -75,13 +78,14 @@
     <parent link="base_footprint"/>
     <child link="base_link"/>
-    <origin xyz="0 0 0" rpy="0 0 -1.5708"/>
+    <origin xyz="0 0 0" rpy="0 0 0"/>
   </joint>
   <link name="base_link">
     <inertial>
-      <origin xyz="0.000129 -0.001817 0.110883"/>
+      <origin xyz="-0.001817 -0.000129 0.110883"/>
       <mass value="14"/>
-      <inertia ixx="1.346868e-01" iyy="4.468661e-02" izz="1.499091e-01" ixy="3.076527e-04" ixz="-2.931603e-05" iyz="2.763693e-05"/>
+      <inertia ixx="4.468661e-02" iyy="1.346868e-01" izz="1.499091e-01" ixy="-3.076527e-04" ixz="2.763693e-05" iyz="2.931603e-05"/>
     </inertial>
     <visual>
+      <origin xyz="0 0 0" rpy="0 0 -1.5708"/>
       <geometry>
         <mesh filename="package://mecanumrover_description/meshes/mecanum3/base_link.stl"
@@ -91,4 +95,5 @@
     </visual>
     <collision>
+      <origin xyz="0 0 0" rpy="0 0 -1.5708"/>
       <geometry>
         <mesh filename="package://mecanumrover_description/meshes/mecanum3/base_link.stl"
@@ -197,24 +202,24 @@
     parent="base_link"
     child="front_left_arm"
-    xyz="-0.085 0.020 0.076"
-    rpy="0 0 ${radians(180)}"/>
+    xyz="0.020 0.085 0.076"
+    rpy="0 0 ${radians(90)}"/>
   <xacro:mecanum_suspension_joint
     name="front_right_suspension_joint"
     parent="base_link"
     child="front_right_arm"
-    xyz="0.085 0.020 0.076"
-    rpy="0 0 ${radians(180)}"/>
+    xyz="0.020 -0.085 0.076"
+    rpy="0 0 ${radians(90)}"/>
   <xacro:mecanum_suspension_joint
     name="back_left_suspension_joint"
     parent="base_link"
     child="back_left_arm"
-    xyz="-0.085 -0.020 0.076"
-    rpy="0 0 0"/>
+    xyz="-0.020 0.085 0.076"
+    rpy="0 0 ${radians(-90)}"/>
   <xacro:mecanum_suspension_joint
     name="back_right_suspension_joint"
     parent="base_link"
     child="back_right_arm"
-    xyz="0.085 -0.020 0.076"
-    rpy="0 0 0"/>
+    xyz="-0.020 -0.085 0.076"
+    rpy="0 0 ${radians(-90)}"/>
   <!-- Wheels -->
   <xacro:mecanum_wheel_rev_link name="front_left_wheel_1"/>
