Commit message: Publish verified ROS 2 Jazzy and Gazebo Harmonic package
Import the qualified package files and use the public Jazzy clone URLs.

File: urdf/g120a.xacro (robot description, xacro)
@@ -4,9 +4,11 @@
   <xacro:include filename="$(find mecanumrover_description)/urdf/materials.xacro" />
   <xacro:include filename="$(find mecanumrover_description)/urdf/g120a.gazebo" />
-  <xacro:include filename="$(find vs_rover_options_description)/urdf/lrf/tg30_g120a.xacro" />
+  <xacro:if value="$(arg use_ros2_control)">
+    <xacro:include filename="$(find mecanumrover_description)/urdf/g120a_ros2_control.xacro" />
+  </xacro:if>
   <!-- OPTION LRF TG30 -->
-  <!-- <xacro:if value="$(arg use_ros2_control)">
-    <xacro:include filename="$(find mecanumrover_description)/urdf/g120a_ros2_control.xacro" />
-  </xacro:if>-->
+  <!-- <xacro:include filename="$(find vs_rover_options_description)/urdf/lrf/tg30_g120a.xacro" /> -->
+  <!-- OPTION BUMPER -->
+  <!-- <xacro:include filename="$(find vs_rover_options_description)/urdf/bumper/bumper_g120a.xacro" /> -->
   <!-- Inertial macros -->
   <xacro:macro name="cylinder_inertial" params="mass radius length">
@@ -130,5 +132,5 @@
       <axis xyz="1 0 0"/>
       <limit lower="-0.1815142" upper="0" effort="300" velocity="20"/>
-      <dynamics damping="5.0" friction="0.1"/>
+      <dynamics damping="10.0" friction="0.1"/>
     </joint>
   </xacro:macro>
@@ -179,4 +181,8 @@
   </xacro:macro>
   <!-- Wheel joint macro -->
+  <!-- Isaac reference motor: 36 V, 7.0 A, rated 7.0 N*m at 250 rpm; peak 18.0 N*m.
+       Reference acceleration: 14.1176470588 rad/s^2; velocity PID: 1.6 / 0.2 / 1.6.
+       Only maximum torque (N*m) and angular velocity (rad/s) below are joint limits.
+       Firmware PID, acceleration ramp and brake switching need controller logic. -->
   <xacro:macro name="g120a_wheel_joint"
                params="name parent child xyz rpy axis_z">
@@ -186,4 +192,5 @@
       <origin xyz="${xyz}" rpy="${rpy}"/>
       <axis xyz="0 0 ${axis_z}"/>
+      <limit effort="18.0" velocity="18.8235294118"/>
     </joint>
   </xacro:macro>

File: urdf/g120a_ros2_control.xacro (robot description, xacro)
@@ -3,5 +3,5 @@
   <ros2_control name="MecanumSystem" type="system">
     <hardware>
-      <plugin>gazebo_ros2_control/GazeboSystem</plugin>
+      <plugin>gz_ros2_control/GazeboSimSystem</plugin>
     </hardware>
     <!-- Wheel joints (velocity) -->

File: urdf/g40a_lb.xacro (robot description, xacro)
@@ -28,5 +28,5 @@
         rpy="${pi/4*rot} 0 ${radians(dir)}"/>
       <axis xyz="0 0 1"/>
-      <dynamics damping="0.001" friction="0.0"/>
+      <dynamics damping="0.0" friction="0.0"/>
     </joint>
     <link name="${prefix}_link">
@@ -141,10 +141,10 @@
   <!-- lrf_mount -->
   <xacro:mecanum_lrf_mount
-    name="front_lrf_mount"
+    name="front_lrf_mount_joint"
     parent="base_link"
     child="front_lrf_mount"
     xyz="0.0 0.0 0.0" rpy="0 0 ${radians(-90)}"/>
     <xacro:mecanum_lrf_mount
-    name="back_lrf_mount"
+    name="back_lrf_mount_joint"
     parent="base_link"
     child="back_lrf_mount"
@@ -184,5 +184,5 @@
       <axis xyz="-1 0 0"/>
       <limit lower="-0.36651914291881" upper="0.10471975511966" effort="10000" velocity="1.0"/>
-      <dynamics damping="630.0" friction="0.0"/>
+      <dynamics damping="8.0" friction="0.0"/>
     </joint>
   </xacro:macro>
@@ -237,4 +237,9 @@
   </xacro:macro>
   <!-- Wheel joint macro -->
+  <!-- Isaac reference motor: 24 V, 3.7 A, rated 2.2 N*m at 270 rpm.
+       Reference acceleration: 17.1428571429 rad/s^2; velocity PID: 1.0 / 0.1 / 1.0.
+       Reference stop-brake torque: 12.0 N*m.
+       Only maximum torque (N*m) and angular velocity (rad/s) below are joint limits.
+       Firmware PID, acceleration ramp and brake switching need controller logic. -->
   <xacro:macro name="mecanum_wheel_joint"
                params="name parent child xyz rpy axis_z">
@@ -244,5 +249,5 @@
       <origin xyz="${xyz}" rpy="${rpy}"/>
       <axis xyz="0 0 ${axis_z}"/>
-      <limit effort="500" velocity="50000"/>
+      <limit effort="3.5" velocity="28.5714285714"/>
       <dynamics damping="0.02"/>
     </joint>

File: urdf/g40a_lb_ros2_control.xacro (robot description, xacro)
@@ -3,5 +3,5 @@
   <ros2_control name="MecanumSystem" type="system">
     <hardware>
-      <plugin>gazebo_ros2_control/GazeboSystem</plugin>
+      <plugin>gz_ros2_control/GazeboSimSystem</plugin>
     </hardware>
 <!-- Wheel joints (velocity) -->

File: urdf/mecanum3.xacro (robot description, xacro)
@@ -9,4 +9,6 @@
   <!-- OPTION LRF TG30 -->
   <!--<xacro:include filename="$(find vs_rover_options_description)/urdf/lrf/tg30_mecanum3.xacro" />-->
+  <!-- OPTION BUMPER -->
+  <!--<xacro:include filename="$(find vs_rover_options_description)/urdf/bumper/bumper_mecanum3.xacro" />-->
   <!-- Inertial macros -->
   <xacro:macro name="cylinder_inertial" params="mass radius length">
@@ -134,5 +136,5 @@
       <axis xyz="1 0 0"/>
       <limit lower="-0.10472" upper="0" effort="300" velocity="20"/>
-      <dynamics damping="5.0" friction="0.1"/>
+      <dynamics damping="8.0" friction="0.1"/>
     </joint>
   </xacro:macro>
@@ -168,4 +170,5 @@
       </inertial>
       <visual>
+        <origin xyz="0 0 0" rpy="0 0 ${radians(-160)}"/>
         <geometry>
           <mesh filename="package://mecanumrover_description/meshes/mecanum3/mecanum_wheel_rev.stl"
@@ -175,4 +178,5 @@
       </visual>
       <collision>
+        <origin xyz="0 0 0" rpy="0 0 ${radians(-160)}"/>
         <geometry>
           <mesh filename="package://mecanumrover_description/meshes/mecanum3/mecanum_wheel_rev.stl"
@@ -183,4 +187,8 @@
   </xacro:macro>
   <!-- Wheel joint macro -->
+  <!-- Isaac reference motor: 24 V, 3.7 A, rated 2.2 N*m at 270 rpm.
+       Reference acceleration: 21.4285714286 rad/s^2; velocity PID: 1.0 / 0.1 / 1.0.
+       Only maximum torque (N*m) and angular velocity (rad/s) below are joint limits.
+       Firmware PID, acceleration ramp and brake switching need controller logic. -->
   <xacro:macro name="mecanum_wheel_joint"
                params="name parent child xyz rpy axis_z">
@@ -190,4 +198,5 @@
       <origin xyz="${xyz}" rpy="${rpy}"/>
       <axis xyz="0 0 ${axis_z}"/>
+      <limit effort="3.5" velocity="28.5714285714"/>
     </joint>
   </xacro:macro>

File: urdf/mecanum3_ros2_control.xacro (robot description, xacro)
@@ -3,5 +3,5 @@
   <ros2_control name="MecanumSystem" type="system">
     <hardware>
-      <plugin>gazebo_ros2_control/GazeboSystem</plugin>
+      <plugin>gz_ros2_control/GazeboSimSystem</plugin>
     </hardware>
     <!-- Wheel joints (velocity) -->
